File: v2/pcb/parrot_v2.brd (EAGLE design)
At the start: 90 x 90 mm, 45 parts, among them Q1 PNO8L07, Q2 PNO8L07, Q3 PNO8L07, Q4 PNO8L07, U1 SHTC3

Commit message: moving along, added pdf, jpg, and png to git lfs
Parts:
- removed C3: 33uf, Seeed-Capacitor:PC-D5.3MM
- removed C_JMP: (no value), SparkFun-Connectors:1X03
- removed C_POT2, NEO_PIX: (no value), con-jst-ph:B3B-PH-K
- removed TP1: EN_test, SparkFun-Connectors:TP_15TH
- removed TP2: PG_test, SparkFun-Connectors:TP_15TH
- removed U$2: TEENSY_3.0_DIL, teensy_3_and_LC:TEENSY_3.0-3.2&LC_DIL
- added C2: 33uf, Seeed-Capacitor:PC-D5.3MM
- added C5, C6: 100nf, adafruit:C2012
- added D5, D6: 1N4004, SparkFun-DiscreteSemi:DIODE-1N4001
- added NEO_PIX1, NEO_PIX2, NEO_PIX3: (no value), con-jst-ph:B3B-PH-K
- added Q5, Q6: PNO8L07, transistor-power:TO220BV
- added R1, R3: 1k, adafruit:M1206
- added R7: 220R, adafruit:M1206
- added SOL5, SOL6: 5566-2, con-molex:5566-2
- added STATUS_LED: B2B-PH-K, con-jst-ph:B2B-PH-K
- added TP10: en_test, SparkFun-Connectors:1X01
- added TP7: neop_test3, SparkFun-Connectors:1X01
- added TP8: neop_test2, SparkFun-Connectors:1X01
- added TP9: neop_test1, SparkFun-Connectors:1X01
- added U$3: TEENSY_3.1-3.2_DIL, teensy_3_and_LC:TEENSY_3.0-3.2&LC_DIL
- C4: value 100nf -> 10uf; device adafruit:C2012 -> Seeed-Capacitor:PC-D5.3MM
- MEMS_L, MEMS_R: value B6B-PH-K -> (none); device con-jst-ph:B6B-PH-K -> SparkFun-Connectors:MOLEX-1X6
- PWR_REG: value S9V11F5S6CMA -> S9V11F5S6CMA_MISSINIG_PINS; device nathans-custom-parts:S9V11F3S5CMA -> nathans-custom-parts:S9V11F3S5CMA_MISSING_PINS
- R10, R11, R2, R4, R5, R6: device SparkFun-Resistors:AXIAL-0.3 -> adafruit:M1206
- TP3, TP4, TP5, TP6: device SparkFun-Connectors:TP_15TH -> SparkFun-Connectors:1X01
- moved MEMS_R 106.6 mm to (21.0, -14.4), turned to 270 degrees
- moved MEMS_L 96.2 mm to (13.2, -14.4), turned to 270 degrees
- moved REG_PWR 75.7 mm to (-32.4, -1.17), turned to 90 degrees
- moved PWR_REG 56.0 mm to (-14.6, -0.66)
- moved TM1 48.8 mm to (-22.9, -26.2), turned to 180 degrees
- moved 12V_IN 47.3 mm to (-21.6, 1.91), flipped to the bottom, turned to 270 degrees
- moved I2C2 46.3 mm to (21.6, -5.13), turned to 270 degrees
- moved TP4 46.1 mm to (-19.1, -24.8), turned to 180 degrees
- moved SOL4 42.6 mm to (0.00, 38.0), turned to 180 degrees
- moved TP6 41.8 mm to (-19.1, -27.3), turned to 180 degrees
- moved I2C1 41.2 mm to (14.6, -5.13), turned to 270 degrees
- moved LDR1 38.9 mm to (-20.4, -32.3)
- moved TM2 38.3 mm to (-15.3, -26.1), turned to 180 degrees
- moved TP3 37.8 mm to (-11.4, -24.8), turned to 180 degrees
- moved TP5 32.3 mm to (-11.4, -27.3), turned to 180 degrees
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Connections:
- removed net BCLK: MEMS_L.3, MEMS_R.3
- removed net I2S_MCLK: U$2.11
- removed net I2S_MISO: U$2.12
- removed net I2S_MOSI: U$2.7
- removed net I2S_RX: U$2.13
- removed net I2S_SCLK: U$2.14/A0
- removed net I2S_SDCS: U$2.10
- removed net I2S_TX: U$2.22/A8
- removed net JMP: C_JMP.2, U$2.6
- removed net LRCLK: MEMS_L.5, MEMS_R.5
- removed net N$15: U$1.GND1
- removed net N$3: PWR_REG.PG, TP2.P$1
- removed net NEO_PIX: NEO_PIX.2, U$2.8
- removed net POT2: C_POT2.2, U$2.17/A3
- new net LED: R7.1, U$3.17/A3
- new net MOT_FAULT: U$1.FAULT, U$3.2
- new net N$1: Q5.G, R5.2
- new net N$2: D5.A, Q5.D, SOL5.2
- new net N$4: Q6.G, R6.2
- new net N$6: D6.A, Q6.D, SOL6.2
- new net N$7: R7.2, STATUS_LED.1
- new net NEO_PIX1: NEO_PIX1.2, TP9.1, U$3.5
- new net NEO_PIX2: NEO_PIX2.2, TP8.1, U$3.8
- new net NEO_PIX3: NEO_PIX3.2, TP7.1, U$3.10
- new net SOL5: R5.1, U$3.4
- new net SOL6: R6.1, U$3.3
- net 12V: now also C2.+, D5.C, D6.C, SOL5.1, SOL6.1; no longer C3.+
- net 3.3V: now also C5.1, R10.2, R11.2, TP3.1, TP4.1, U$3.3.3V; no longer C4.2, C_JMP.1, C_POT2.1, R10.P$2, R11.P$2, TP3.P$1, TP4.P$1, U$2.3.3V
- net 5V: now also C4.+, C6.1, NEO_PIX1.1, NEO_PIX2.1, NEO_PIX3.1, U$3.VIN; no longer NEO_PIX.1, U$2.VIN
- net AGND: now also U$3.AGND; no longer C_POT2.3, U$2.AGND
- net GND: now also C2.-, C4.-, C5.2, C6.2, NEO_PIX1.3, NEO_PIX2.3, NEO_PIX3.3, Q5.S, Q6.S, REG_PWR.1, STATUS_LED.2, U$1.GND1, U$3.GND; no longer C3.-, C4.1, C_JMP.3, NEO_PIX.3, REG_PWR.2, U$2.GND
- net I2S_BCLK: now also MEMS_L.3, MEMS_R.3, U$3.9; no longer U$2.9
- net I2S_DATA: now also U$3.13
- net I2S_LRCLK: now also MEMS_L.5, MEMS_R.5, U$3.23/A9; no longer U$2.23/A9
- net LDR1: now also TM1.3, TP6.1, U$3.15/A1; no longer TP6.P$1
- net LDR2: now also TM2.3, TP5.1, U$3.16/A2; no longer TP5.P$1
- net MOT_COAST: now also U$3.20/A6; no longer U$2.21/A7
- net MOT_DIR: now also U$3.21/A7; no longer U$2.20/A6
- net MOT_SPEED: now also U$3.22/A8; no longer U$2.15/A1
- net N$10: now also REG_PWR.2, TP10.1; no longer REG_PWR.1, TP1.P$1
- net N$11: now also R3.2; no longer R5.P$2
- net N$13: now also R4.2; no longer R6.P$2
- net N$24: now also R1.2; no longer R2.P$2
- net N$5: now also R2.2; no longer R4.P$2
- net POT1: now also U$3.14/A0; no longer U$2.16/A2
- net SCL0: now also R11.1, U$3.19/A5; no longer R11.P$1, U$2.19/A5
- net SDA0: now also R10.1, U$3.18/A4; no longer R10.P$1, U$2.18/A4
- net SOL1: now also R1.1, U$3.12; no longer R2.P$1, U$2.2
- net SOL2: now also R2.1, U$3.11; no longer R4.P$1, U$2.3
- net SOL3: now also R3.1, U$3.7; no longer R5.P$1, U$2.4
- net SOL4: now also R4.1, U$3.6; no longer R6.P$1, U$2.5
Routing:
- net 5V: track 25.6 -> 112.9 mm
- net I2S_DATA: track 0.00 -> 52.1 mm
- net NEO_PIX: track 51.3 -> 0.00 mm
- net SOL6: track 0.00 -> 49.3 mm
- net SOL5: track 0.00 -> 47.4 mm
- net N$7: track 0.00 -> 41.9 mm
- net LDR1: track 7.65 -> 47.0 mm
- net NEO_PIX1: track 0.00 -> 35.3 mm
- net LDR2: track 8.40 -> 42.4 mm
- net I2S_MISO: track 32.7 -> 0.00 mm
- net SOL4: track 3.24 -> 35.8 mm
- net I2S_MCLK: track 32.5 -> 0.00 mm
- net MOT_DIR: track 36.7 -> 5.92 mm
- net NEO_PIX2: track 0.00 -> 30.2 mm
- net MOT_COAST: track 34.5 -> 5.85 mm
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- added copper zone on layer 1, net 12V
Other:
- board text added: "12V"
- board text added: "BCL"
- board text added: "DI"
- board text added: "LR"
- board text added: "Lyre Genus Mainboard v2.0"
- board text removed: "+"
- board text removed: "-"
- board text removed: "COAST"
- board text removed: "I2S"
- board text removed: "M1"
- board text removed: "M2"
- board text removed: "Neo Pixels"
- board text removed: "PG"
- board text removed: "Parrot Genus Mainboard v1.1"
- board text removed: "VIN"
- board text removed: "VM"
- board text removed: "VOUT"
