File: pcb/eye_stocks/lyre_eye_stocks_40mm_breakout.brd (EAGLE design)
At the start: 40.1 x 40.1 mm, 36 parts, among them P1 B10B-PH-K, U1 SHTC3, U2 VEML6030-GS15

Commit message: updated some long needed things for the repo
Parts:
- removed L/R_SEL: (no value), SparkFun-Connectors:1X03
- added JP1, JP3: JUMPER-SMT_3_1-NC_TRACE_SILK, SparkFun-Jumpers:SMT-JUMPER_3_1-NC_TRACE_SILK
- added JP4: JUMPER-SMT_2_NO_SILK, SparkFun-Jumpers:SMT-JUMPER_2_NO_SILK
- NC1, NC10, NC2, NC3, NC4, NC5, NC6, NC7, NC8, NC9: device rcl:C0805K -> rcl:C0805
- NEO_01, NEO_02, NEO_03, NEO_04, NEO_05, NEO_06, NEO_07, NEO_08, NEO_09, NEO_10: value WS2812B5050 -> WS2812; device adafruit:WS2812B -> WS2812B:WS2812B
- R15: device adafruit:M0805 -> PulseOximeterECG_AU:R0805
- R3, R5, R6: device audio amplifier example:R0805 -> PulseOximeterECG_AU:R0805
- moved C1 0.73 mm to (-0.16, -2.81), turned to 0 degrees
- moved VEML_F 0.43 mm to (-3.93, -3.16)
Connections:
- new net NIN: JP1.2, P1.4
- net 3.3V: now also JP3.3; no longer L/R_SEL.3
- net GND: now also JP3.1; no longer L/R_SEL.1
- net N$2: now also JP1.1
- net N$6: now also JP3.2; no longer L/R_SEL.2
- net NEOP_IN: now also JP1.3, JP4.2; no longer P1.4
- net NEOP_OUT: now also JP4.1
Routing:
- net NIN: track 0.00 -> 26.2 mm, vias 0 -> 3
- net NEOP_OUT: track 18.4 -> 37.3 mm, vias 0 -> 1
- net NEOP_IN: track 13.2 -> 28.5 mm, vias 0 -> 2
- net N$2: track 12.9 -> 20.9 mm
- net GND: track 30.7 -> 35.0 mm
- net N$6: track 5.69 -> 8.96 mm
- net 3.3V: track 47.1 -> 50.2 mm
- net LRCLK: track 12.6 -> 10.2 mm
- net N$1: track 19.2 -> 20.6 mm
- net SDA0: track 32.1 -> 31.0 mm
- net BCLK: track 12.9 -> 12.3 mm
- net SCL0: track 20.9 -> 20.3 mm
- net 5V: track 133.9 -> 133.6 mm, vias 7 -> 8
Other:
- board text added: "0.1uF"
- board text added: "3.3v"
- board text added: "5v"
- board text added: "BCLK"
- board text added: "DIN"
- board text added: "F"
- board text added: "GND"
- board text added: "ID#"
- board text added: "L"
- board text added: "LRCLK"
- board text added: "Lyre Eye-Stocks Rev 1.2"
- board text added: "NEOP"
- board text added: "NeoIn"
- board text added: "NeoOut"
- board text added: "R"
- board text added: "SCL"
- board text added: "SDA"
- board text added: "channel"
- board text removed: "Designed by Nathan Villicana-Shaw 2020"
- board text removed: "ID #"
- board text removed: "Left"
- board text removed: "Lyre Eye-Stocks Rev 1.1"
- board text removed: "Right"
