File: pcb/eye_stocks/lyre_eye_stocks_40mm_breakout.sch (EAGLE design)
At the start: 36 parts, among them P1 B10B-PH-K, U1 SHTC3, U2 VEML6030-GS15

Commit message: updated some long needed things for the repo
Parts:
- removed L/R_SEL: (no value), SparkFun-Connectors:CONN_03
- added JP1, JP3: JUMPER-SMT_3_1-NC_TRACE_SILK, SparkFun-Jumpers:JUMPER-SMT_3_1-NC_TRACE_SILK
- added JP4: JUMPER-SMT_2_NO_SILK, SparkFun-Jumpers:JUMPER-SMT_2_NO_SILK
- NC1, NC10, NC2, NC3, NC4, NC5, NC6, NC7, NC8, NC9: device rcl:C-USC0805K -> rcl:C-USC0805
- NEO_01, NEO_02, NEO_03, NEO_04, NEO_05, NEO_06, NEO_07, NEO_08, NEO_09, NEO_10: value WS2812B5050 -> WS2812; device adafruit:WS2812B5050 -> WS2812B:WS2812
- R15: device adafruit:R-US_M0805 -> PulseOximeterECG_AU:R-US_R0805
- R3, R5, R6: device audio amplifier example:R-US_R0805 -> PulseOximeterECG_AU:R-US_R0805
Connections:
- new net NIN: JP1.2, P1.4
- net 3.3V: now also JP3.3; no longer L/R_SEL.3
- net GND: now also JP3.1; no longer L/R_SEL.1
- net N$2: now also JP1.1
- net N$6: now also JP3.2; no longer L/R_SEL.2
- net NEOP_IN: now also JP1.3, JP4.2; no longer P1.4
- net NEOP_OUT: now also JP4.1
Other:
- note added: "JST-ph Connector"
- note added: "NeoPixel LEDs (bottom)"
- note added: "NeoPixel LEDs (top)"
- note removed: "14/10/2019"
- note removed: "Designed by Nathan Villicana-Shaw Victoria University of Wellington School of Engineering and Computer Science"
- note removed: "NeoPixel LEDs"
- moved on the sheet: C1, C2, C3, C4, C8, C9, MK_REAR, NC10, NC6, NC7, NC8, NC9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
