File: pcb/v0_2/parrot_v2.brd (EAGLE design)
At the start: 90 x 90 mm, 59 parts, among them Q1 PNO8L07, Q2 PNO8L07, Q3 PNO8L07, Q4 PNO8L07, Q5 PNO8L07, Q6 PNO8L07, U1 SHTC3

Commit message: updated some long needed things for the repo
Other:
- board text added: "Explorator Mainboard v0.2"
- board text removed: "Lyre Genus Mainboard v2.0"
Changed lines of the file:
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@@
 <?xml version="1.0" encoding="utf-8"?>
 <!DOCTYPE eagle SYSTEM "eagle.dtd">
-<eagle version="9.5.1">
+<eagle version="9.6.2">
 <drawing>
 <settings>
-<setting alwaysvectorfont="yes"/>
+<setting alwaysvectorfont="no"/>
 <setting verticaltext="up"/>
 </settings>
@@
 <layer number="14" name="Route14" color="1" fill="6" visible="no" active="no"/>
 <layer number="15" name="Route15" color="4" fill="6" visible="no" active="no"/>
-<layer number="16" name="Bottom" color="1" fill="1" visible="yes" active="yes"/>
+<layer number="16" name="Bottom" color="1" fill="1" visible="no" active="yes"/>
 <layer number="17" name="Pads" color="2" fill="1" visible="yes" active="yes"/>
 <layer number="18" name="Vias" color="2" fill="1" visible="yes" active="yes"/>
-<layer number="19" name="Unrouted" color="6" fill="1" visible="yes" active="yes"/>
+<layer number="19" name="Unrouted" color="6" fill="1" visible="no" active="yes"/>
 <layer number="20" name="Dimension" color="24" fill="1" visible="yes" active="yes"/>
 <layer number="21" name="tPlace" color="7" fill="1" visible="yes" active="yes"/>
-<layer number="22" name="bPlace" color="7" fill="1" visible="yes" active="yes"/>
-<layer number="23" name="tOrigins" color="15" fill="1" visible="yes" active="yes"/>
-<layer number="24" name="bOrigins" color="15" fill="1" visible="yes" active="yes"/>
+<layer number="22" name="bPlace" color="7" fill="1" visible="no" active="yes"/>
+<layer number="23" name="tOrigins" color="15" fill="1" visible="no" active="yes"/>
+<layer number="24" name="bOrigins" color="15" fill="1" visible="no" active="yes"/>
 <layer number="25" name="tNames" color="7" fill="1" visible="yes" active="yes"/>
-<layer number="26" name="bNames" color="7" fill="1" visible="yes" active="yes"/>
+<layer number="26" name="bNames" color="7" fill="1" visible="no" active="yes"/>
 <layer number="27" name="tValues" color="7" fill="1" visible="no" active="yes"/>
 <layer number="28" name="bValues" color="7" fill="1" visible="no" active="yes"/>
@@
 <layer number="38" name="bTest" color="7" fill="1" visible="no" active="yes"/>
 <layer number="39" name="tKeepout" color="4" fill="11" visible="yes" active="yes"/>
-<layer number="40" name="bKeepout" color="1" fill="11" visible="yes" active="yes"/>
+<layer number="40" name="bKeepout" color="1" fill="11" visible="no" active="yes"/>
 <layer number="41" name="tRestrict" color="4" fill="10" visible="yes" active="yes"/>
-<layer number="42" name="bRestrict" color="1" fill="10" visible="yes" active="yes"/>
+<layer number="42" name="bRestrict" color="1" fill="10" visible="no" active="yes"/>
 <layer number="43" name="vRestrict" color="2" fill="10" visible="no" active="yes"/>
 <layer number="44" name="Drills" color="7" fill="1" visible="no" active="yes"/>
@@
 <layer number="50" name="dxf" color="7" fill="1" visible="no" active="no"/>
 <layer number="51" name="tDocu" color="7" fill="1" visible="yes" active="yes"/>
-<layer number="52" name="bDocu" color="7" fill="1" visible="yes" active="yes"/>
+<layer number="52" name="bDocu" color="7" fill="1" visible="no" active="yes"/>
 <layer number="53" name="tGND_GNDA" color="7" fill="1" visible="no" active="no"/>
 <layer number="54" name="bGND_GNDA" color="7" fill="1" visible="no" active="no"/>
@@
 </layers>
 <board>
-<fusionsync huburn="a.cGVyc29uYWw6dWUyYWRjZTVi" projecturn="a.cGVyc29uYWw6dWUyYWRjZTViIzIwMTkwNTE2MTk0MjIzODUx" f3durn="urn:adsk.wipprod:dm.lineage:NFP_iIeHQGms001mJm5pbg" pcbguid="0bd6a69f-3b44-4c63-bd4f-b1bf585d3a3a" lastpulledtime="" lastsyncedchangeguid="00897717-f45c-77c2-13a5-944085ebe09b"/>
+<fusionsync huburn="a.cGVyc29uYWw6dWUyYWRjZTVi" projecturn="a.cGVyc29uYWw6dWUyYWRjZTViIzIwMTkwNTE2MTk0MjIzODUx" f3durn="urn:adsk.wipprod:dm.lineage:NFP_iIeHQGms001mJm5pbg" pcbguid="0bd6a69f-3b44-4c63-bd4f-b1bf585d3a3a" lastpulledtime="" lastsyncedchangeguid="00897717-f45c-77c2-13a5-944085ebe09b" latestrevisionid="" lastsyncedrevisionid="" lastboardhashguid="" lastpushedtime="" linktopcb3d="false"/>
 <plain>
 <circle x="0" y="0" radius="45" width="0.0762" layer="20"/>
-<text x="22.19325" y="-33.3121" size="1.778" layer="25" rot="R180">Lyre Genus
-Mainboard v2.0</text>
+<text x="22.19325" y="-33.3121" size="1.778" layer="25" rot="R180">Explorator
+Mainboard v0.2</text>
 <text x="18.3388" y="-38.0746" size="1.016" layer="25" rot="R180">designed by
 Nathan Villicana-Shaw</text>
@@
 <contactref element="U1" pad="5"/>
 <polygon width="0.8128" layer="16">
-<vertex x="-45.72" y="45.72"/>
-<vertex x="45.72" y="45.72"/>
-<vertex x="45.72" y="-32.385"/>
-<vertex x="-45.72" y="-32.385"/>
+<vertex x="19.628740625" y="-32.385"/>
+<vertex x="-21.6310875" y="-32.385" curve="-90"/>
+<vertex x="-45.72" y="-8.2960875"/>
+<vertex x="-45.72" y="-0.347059375" curve="-90"/>
+<vertex x="0.347059375" y="45.72" curve="-90"/>
+<vertex x="45.72" y="0.347059375"/>
+<vertex x="45.72" y="-6.293740625" curve="-90"/>
 </polygon>
 <contactref element="PWR_REG" pad="GND"/>
@@
 <vertex x="46.0248" y="6.096"/>
 <vertex x="46.1264" y="6.1976"/>
-<vertex x="46.1264" y="-21.4376"/>
-<vertex x="34.7472" y="-32.8168"/>
-<vertex x="-33.4264" y="-32.8168"/>
-<vertex x="-44.8056" y="-21.4376"/>
-<vertex x="-45.4152" y="-20.828"/>
+<vertex x="46.1264" y="-13.754328125" curve="-45"/>
+<vertex x="40.69350625" y="-26.87049375" curve="-45.000009"/>
+<vertex x="26.337853125" y="-32.8168"/>
+<vertex x="-24.080734375" y="-32.8168" curve="-45"/>
+<vertex x="-40.034784375" y="-26.208415625" curve="-45.21622"/>
+<vertex x="-45.38659375" y="-13.2187375"/>
 <vertex x="-45.3136" y="6.1976"/>
 </polygon>
@@
 <wire x1="-25.677" y1="-10.2386" x2="-25.677" y2="-10.2362" width="1.524" layer="1"/>
 <wire x1="-19.7892" y1="-0.79" x2="-19.7892" y2="-5.9716" width="1.524" layer="1"/>
-<polygon width="0.8128" layer="1">
-<vertex x="-45.5422" y="9.8806" curve="90"/>
-<vertex x="-45.5168" y="9.8552"/>
-</polygon>
 <wire x1="-25.6794" y1="-10.2362" x2="-25.654" y2="-10.2616" width="1.27" layer="1"/>
 <polygon width="0.762" layer="1">
-<vertex x="-45.72" y="45.72"/>
+<vertex x="46.0248" y="9.8552" curve="90.036474"/>
+<vertex x="10.46474375" y="45.595696875"/>
+<vertex x="-12.293528125" y="45.646046875" curve="90.300423"/>
 <vertex x="-45.6184" y="12.2936"/>
 <vertex x="-23.4696" y="12.2936" curve="-90"/>
@@
 <vertex x="25.7048" y="9.652"/>
 <vertex x="45.8216" y="9.652" curve="90"/>
-<vertex x="46.0248" y="9.8552"/>
-<vertex x="46.1264" y="45.5168"/>
 </polygon>
 </signal>
