File: pcb/v0_2/parrot_v2.sch (EAGLE design)
At the start: 59 parts, among them Q1 PNO8L07, Q2 PNO8L07, Q3 PNO8L07, Q4 PNO8L07, Q5 PNO8L07, Q6 PNO8L07, U1 SHTC3

Commit message: updated some long needed things for the repo
Other:
- note added: "2019"
- note added: "Explorator v0.2"
- note added: "Nathan Daniel Villicana-Shaw"
- note removed: "(test two neoP channels, along with the motor driver and audio all running at same time...)"
- note removed: "Add Test Ponts for I2C, I2S, and other things..."
- note removed: "Add one more connector for I2C"
- note removed: "Add second NeoP channel"
- note removed: "Add some cable cut-out slots on outside where no traces are"
- note removed: "Fix Silkscreen side for the Solenoids and Motor Outputs"
- note removed: "Make sure this cap is placed with correct polarity"
- note removed: "Perhaps replace the JST ph connectors for the microphone boards to the onboard footprints"
- note removed: "Switch side that the NeoPixels connectors/silkscreen is on"
- note removed: "Test is the MEMS microphones will work onboard or if they need to be off-board"
- note removed: "add Status LED"
- note removed: "input selector for 5v and 12v on solenoid outputs"
- note removed: "replace 0.3 with 1206 components"
- note removed: "replace all test points with 0.1" pads"
- moved on the sheet: C5, U1
