File: pcb/v1/lyre_v1.brd (EAGLE design)
At the start: 99 x 99 mm, 74 parts, among them M1 5566-2, M2 5566-2, M3 5566-2, Q1 PNO8L07, Q2 PNO8L07, Q3 PNO8L07, Q4 PNO8L07, Q5 PNO8L07, Q6 PNO8L07, Q7 PNO8L07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

Commit message: updated some long needed things for the repo
Changed lines of the file:
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@@
 <?xml version="1.0" encoding="utf-8"?>
 <!DOCTYPE eagle SYSTEM "eagle.dtd">
-<eagle version="9.6.1">
+<eagle version="9.6.2">
 <drawing>
 <settings>
-<setting alwaysvectorfont="yes"/>
+<setting alwaysvectorfont="no"/>
 <setting verticaltext="up"/>
 </settings>
@@
 <layer number="25" name="tNames" color="7" fill="1" visible="yes" active="yes"/>
 <layer number="26" name="bNames" color="7" fill="1" visible="yes" active="yes"/>
-<layer number="27" name="tValues" color="7" fill="1" visible="yes" active="yes"/>
-<layer number="28" name="bValues" color="7" fill="1" visible="yes" active="yes"/>
+<layer number="27" name="tValues" color="7" fill="1" visible="no" active="yes"/>
+<layer number="28" name="bValues" color="7" fill="1" visible="no" active="yes"/>
 <layer number="29" name="tStop" color="7" fill="3" visible="no" active="yes"/>
 <layer number="30" name="bStop" color="7" fill="6" visible="no" active="yes"/>
@@
 Nathan Villicana-Shaw</text>
 <text x="-33.6692" y="-32.41805" size="1.016" layer="25" rot="R135">2020</text>
-<text x="40.16375" y="-66.00825" size="1.016" layer="27" ratio="16" rot="R180">3.3V</text>
 <circle x="-26.86685" y="26.8478" radius="4.869228125" width="0.1524" layer="21"/>
 <circle x="26.85415" y="26.8478" radius="5.1481" width="0.1524" layer="21"/>
@@
 <contactref element="BUT4" pad="2"/>
 <polygon width="1.27" layer="16">
-<vertex x="-55.88" y="53.34"/>
-<vertex x="-55.88" y="-50.8"/>
-<vertex x="58.42" y="-50.8"/>
-<vertex x="58.42" y="53.34"/>
+<vertex x="49.911" y="-1.04919375"/>
+<vertex x="49.911" y="-0.476821875" curve="90"/>
+<vertex x="-0.603821875" y="50.038"/>
+<vertex x="-1.788109375" y="50.038" curve="90"/>
+<vertex x="-49.911" y="1.915109375"/>
+<vertex x="-49.911" y="0.714203125" curve="90"/>
+<vertex x="0.460203125" y="-49.657"/>
+<vertex x="1.30319375" y="-49.657" curve="90"/>
 </polygon>
 <wire x1="0.239" y1="17.91" x2="0.239" y2="21.13435" width="1.27" layer="1"/>
@@
 <wire x1="-19.92029375" y1="18.919703125" x2="-20.096534375" y2="18.74206875" width="1.27" layer="1"/>
 <polygon width="1.27" layer="1">
-<vertex x="-59.69" y="55.118"/>
-<vertex x="-59.69" y="-52.578"/>
-<vertex x="61.722" y="-52.578"/>
-<vertex x="61.722" y="55.118"/>
+<vertex x="50.038" y="-1.037171875"/>
+<vertex x="50.038" y="-0.783171875" curve="90"/>
+<vertex x="-0.910171875" y="50.165" curve="90"/>
+<vertex x="-49.657" y="1.418171875" curve="90"/>
+<vertex x="1.418171875" y="-49.657" curve="90"/>
 </polygon>
 <wire x1="7.859" y1="-15.11" x2="6.967" y2="-16.002" width="1.27" layer="16"/>
@@
 <wire x1="39.65039375" y1="-21.511096875" x2="39.49156875" y2="-21.289" width="2.54" layer="1"/>
 <wire x1="-24.157128125" y1="-21.469278125" x2="-24.157128125" y2="-17.842871875" width="1.27" layer="16"/>
-<wire x1="-24.157128125" y1="-17.842871875" x2="-28" y2="-14" width="1.27" layer="16"/>
-<wire x1="-28" y1="-14" x2="-31.0926875" y2="-14" width="1.27" layer="16"/>
-<wire x1="-31.0926875" y1="-14" x2="-31.654490625" y2="-14.561803125" width="1.27" layer="16"/>
-<wire x1="-28" y1="-14" x2="-35.553815625" y2="-6.446184375" width="1.27" layer="16"/>
+<wire x1="-24.157128125" y1="-17.842871875" x2="-29.524" y2="-12.476" width="1.27" layer="16"/>
+<wire x1="-29.524" y1="-12.476" x2="-29.5686875" y2="-12.476" width="1.27" layer="16"/>
+<wire x1="-29.5686875" y1="-12.476" x2="-31.654490625" y2="-14.561803125" width="1.27" layer="16"/>
+<wire x1="-29.524" y1="-12.476" x2="-35.553815625" y2="-6.446184375" width="1.27" layer="16"/>
 <wire x1="-35.553815625" y1="-6.446184375" x2="-35.553815625" y2="-2.213959375" width="1.27" layer="16"/>
 <wire x1="-35.553815625" y1="-2.213959375" x2="-35.553815625" y2="9.347584375" width="1.27" layer="16"/>
-<wire x1="-33.7798" y1="13.818203125" x2="-30.192378125" y2="20.096190625" width="1.27" layer="16"/>
-<wire x1="-33.7798" y1="11.9068" x2="-33.7798" y2="13.818203125" width="1.27" layer="16"/>
+<wire x1="-34.118465625" y1="13.2255375" x2="-30.192378125" y2="20.096190625" width="1.27" layer="16"/>
 <wire x1="-30.192378125" y1="20.096190625" x2="-28.788965625" y2="21.96740625" width="1.27" layer="16"/>
 <wire x1="-28.788965625" y1="21.96740625" x2="-26.756371875" y2="24" width="1.27" layer="16"/>
@@
 <wire x1="-23.864203125" y1="24" x2="-22.932103125" y2="24.9321" width="1.27" layer="16"/>
 <wire x1="-22.932103125" y1="24.9321" x2="-17.094271875" y2="30.76993125" width="1.27" layer="16"/>
-<wire x1="-35.553815625" y1="9.347584375" x2="-33.372065625" y2="11.529334375" width="1.27" layer="16"/>
-<wire x1="-32.849" y1="10.976" x2="-33.7798" y2="11.9068" width="1.27" layer="16"/>
 <wire x1="-26.756371875" y1="24" x2="-23.864203125" y2="24" width="1.27" layer="16"/>
 <wire x1="-3.002828125" y1="36.115909375" x2="-2.333903125" y2="36.34305625" width="1.27" layer="16"/>
@@
 <wire x1="-3.885575" y1="36.115909375" x2="-3.002828125" y2="36.115909375" width="1.27" layer="16"/>
 <wire x1="-2.333903125" y1="36.34305625" x2="3.199296875" y2="36.34305625" width="1.27" layer="16"/>
-<wire x1="3.199296875" y1="36.34305625" x2="7.546584375" y2="31.99576875" width="1.27" layer="16"/>
-<wire x1="7.546584375" y1="31.99576875" x2="9.65246875" y2="31.99576875" width="1.27" layer="16"/>
+<wire x1="7.546584375" y1="31.99576875" x2="3.199296875" y2="36.34305625" width="1.27" layer="16"/>
 <wire x1="10.7204125" y1="33.1129" x2="10.7204125" y2="33.0637125" width="1.27" layer="16"/>
-<wire x1="10.7204125" y1="33.0637125" x2="9.65246875" y2="31.99576875" width="1.27" layer="16"/>
 <wire x1="10.7204125" y1="33.1129" x2="10.8537625" y2="32.97955" width="1.27" layer="16"/>
-<wire x1="10.8537625" y1="32.97955" x2="10.8537625" y2="28.187365625" width="1.27" layer="16"/>
 <wire x1="21.33126875" y1="22.138184375" x2="10.8537625" y2="28.187365625" width="1.27" layer="16"/>
 <wire x1="22.746903125" y1="22.397153125" x2="22.487934375" y2="22.138184375" width="1.27" layer="16"/>
@@
 <wire x1="-0.98286875" y1="35.12475625" x2="-0.98286875" y2="28.956" width="1.524" layer="1"/>
 <wire x1="-21.85323125" y1="23.862775" x2="-22.932103125" y2="24.9321" width="1.27" layer="16"/>
-<wire x1="-32.8077" y1="11.0436625" x2="-33.372065625" y2="11.529334375" width="1.27" layer="16"/>
 <wire x1="43.96221875" y1="-6.69053125" x2="43.5594" y2="-6.69053125" width="1.27" layer="16"/>
 <wire x1="43.5594" y1="-6.69053125" x2="42.291684375" y2="-7.958246875" width="1.27" layer="16"/>
@@
 <wire x1="-17.90299375" y1="23.9084875" x2="-17.927959375" y2="23.862775" width="1.27" layer="16"/>
 <wire x1="-17.927959375" y1="23.862775" x2="-21.85323125" y2="23.862775" width="1.27" layer="16"/>
+<wire x1="10.8537625" y1="28.187365625" x2="8.2175625" y2="30.823565625" width="1.27" layer="16"/>
+<wire x1="8.2175625" y1="30.823565625" x2="7.546584375" y2="31.49454375" width="1.27" layer="16"/>
+<wire x1="7.546584375" y1="31.49454375" x2="7.546584375" y2="31.99576875" width="1.27" layer="16"/>
+<wire x1="10.7204125" y1="33.1129" x2="8.431078125" y2="30.823565625" width="1.27" layer="16"/>
+<wire x1="8.431078125" y1="30.823565625" x2="8.2175625" y2="30.823565625" width="1.27" layer="16"/>
+<wire x1="-35.553815625" y1="9.347584375" x2="-35.426815625" y2="9.474584375" width="1.27" layer="16"/>
+<wire x1="-35.426815625" y1="11.9171875" x2="-35.426815625" y2="10.922" width="1.27" layer="16"/>
+<wire x1="-35.426815625" y1="10.922" x2="-35.426815625" y2="9.474584375" width="1.27" layer="16"/>
+<wire x1="-35.426815625" y1="11.9171875" x2="-34.118465625" y2="13.2255375" width="1.27" layer="16"/>
+<wire x1="-32.8077" y1="11.0436625" x2="-35.305153125" y2="11.0436625" width="1.27" layer="16"/>
+<wire x1="-35.305153125" y1="11.0436625" x2="-35.426815625" y2="10.922" width="1.27" layer="16"/>
 </signal>
 <signal name="5V">
