File: pcb/v1/lyre_v1.sch (EAGLE design)
At the start: 74 parts, among them M1 5566-2, M2 5566-2, M3 5566-2, Q1 PNO8L07, Q2 PNO8L07, Q3 PNO8L07, Q4 PNO8L07, Q5 PNO8L07, Q6 PNO8L07, Q7 PNO8L07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

Commit message: updated some long needed things for the repo
Other:
- note added: "Solenoids"
- note removed: "Add decoupling caps for teensy"
- note removed: "LDRs are not connected!!!!!!"
- note removed: "Make sure this cap is placed with correct polarity"
- note removed: "Perhaps replace the JST ph connectors for the microphone boards to the onboard footprints"
- note removed: "Test is the MEMS microphones will work onboard or if they need to be off-board"
- note removed: "add fault for the motor driver"
- moved on the sheet: I2C2, I2S, M1-1, M1-2, M2-1, M2-2, M3-1, M3-2, MOT1, MOT2, MOT3
